Commit message: Manos: q=0 es la mano abierta y el limite superior la mano cerrada
Los ceros y limites de las 12 juntas de cada mano se fijan ahora desde el
manual de usuario de la RH56DFTP, apartado 2.6.11 (paginas impresas 21 y 22),
que define un angulo de cuerda por DOF contra el plano metacarpiano:

  dedos            alpha   176 (abierto) -> 20 (cerrado)
  pulgar flexion   theta    70           -> -13
  pulgar rotacion  beta    165           -> 90

No son angulos articulares, asi que se calcularon sobre el modelo y se
resolvio que valor de q produce cada extremo. Cada origen de junta se giro
para que q=0 caiga exactamente en el angulo de abierto, y el limite superior
en el de cerrado:

  junta          giro del cero     q_max (rad)
  index_1          -1.32 deg        1.60795
  middle_1         -1.73 deg        1.59037
  ring_1           -1.56 deg        1.60951
  little_1         -0.44 deg        1.67173
  thumb_1          +1.85 deg        1.06242
  thumb_swing     +12.85 deg        1.30900

Las cuatro q_max de los dedos difieren porque cada dedo asienta en la palma
con su propio angulo, de modo que el mismo barrido 176..20 cuesta un recorrido
articular algo distinto. Las mimic llevan multiplicador * q_max y su cero se
giro multiplicador * delta, o la falange distal no quedaria en su sitio con
q=0.

Ningun eje cambia: los seis cierran al crecer q. Con eso el mapeo al SDK es
uno solo para los seis:

  ANGLE_SET = 1000 * (1 - q / q_max)

Dos correcciones de camino, ambas detectadas al contrastar con el modelo:

- Una medida intermedia tomaba beta como angulo 3D contra la normal de la
  palma, cuando la figura del manual es una vista superior y hay que proyectar
  al plano x-y. Esa medida hacia creer que el swing del pulgar corria invertido
  respecto a los otros cinco DOF y que habia que voltear su eje. No es asi:
  beta decrece con q como los demas. El usuario lo detecto en RViz, donde
  swing=1.5331 se ve como beta~90 y swing=0 como beta~180, que es justo lo que
  da la definicion correcta (90.0 y 177.8).
- El primer calculo de los limites superiores tomaba la yema como el vertice
  mas lejano en cada configuracion, que cambia al curvarse el dedo, en vez de
  un punto material fijo. Daba extremos pasados de 3.5 a 5 grados.

Verificacion:
  los 12 extremos sobre el modelo    error maximo 4.6e-05 grados
  simetria izq/der, misma consigna   0.000000 mm en abierta, cerrada y 2 aleatorias
  autocolision al cierre total       los 4 dedos ya no tocan la palma (antes el
                                     medio penetraba 0.51 mm); solo el pulgar
                                     apoya, 2.78 mm contra la palma y 0.37 mm
                                     contra el indice
  XML 9/9, xacro 3/3, check_urdf 6/6, nq=46 nv=45, masa 68.6640 kg

Comprobado ademas visualmente en RViz con display_h1_2_with_hands.launch.py:
a q=0 los cuatro dedos quedan casi rectos y el pulgar abierto, y a q_max la
mano cierra en puno con el pulgar encima.

Se propagan el espejo a la mano derecha y los dos URDF planos; h1_2_handless
no se toca porque no lleva manos.

Co-Authored-By: Claude Opus 5 <noreply@anthropic.com>
Claude-Session: https://claude.ai/code/session_01WDAX8VZbrLhjdUkohUZLGo

File: ros_h1_2_ws/src/h1_2_inspire_description/urdf/h1_2_hands_isaac.urdf (robot description, URDF)
Before this commit: robot h1_2_with_inspire_hands, 58 links, 57 joints
Joints:
- joint left_index_1_joint: limit lower=0 upper=1.6 effort=1 velocity=100 -> lower=0 upper=1.60795403606 effort=1 velocity=100; origin xyz=-0.048156 0.11125 0.045404 rpy=1.6057 0 -1.5708 -> xyz=-0.048156 0.11125 0.045404 rpy=1.60570928804 -0.0230624359379 -1.57160543366
- joint left_index_2_joint: limit lower=0 upper=1.6 effort=1 velocity=100 -> lower=0 upper=1.68835173786 effort=1 velocity=100; origin xyz=0.00259487212105013 0.0326721877470773 -0.000299999999999988 rpy=0 0 0 -> xyz=0.00259487212105013 0.0326721877470773 -0.000299999999999988 rpy=0 -0 0.0242303183457
- joint left_little_1_joint: limit lower=0 upper=1.6 effort=1 velocity=100 -> lower=0 upper=1.67172785459 effort=1 velocity=100; origin xyz=0.016446 0.11125 0.042817 rpy=1.4661 0 -1.5708 -> xyz=0.016446 0.11125 0.042817 rpy=1.46609698912 -0.00756999419343 -1.57000452558
- joint left_little_2_joint: limit lower=0 upper=1.6 effort=1 velocity=100 -> lower=0 upper=1.75531424732 effort=1 velocity=100; origin xyz=0.0023072 0.032694 -0.0003 rpy=0 0 0 -> xyz=0.0023072 0.032694 -0.0003 rpy=0 -0 0.00799225759443
- joint left_middle_1_joint: limit lower=0 upper=1.6 effort=1 velocity=100 -> lower=0 upper=1.590368352 effort=1 velocity=100; origin xyz=-0.026577 0.11125 0.046044 rpy=1.5708 0 -1.5708 -> xyz=-0.026577 0.11125 0.046044 rpy=1.57080000168 -0.0302474957799 -1.57080011114
- joint left_middle_2_joint: limit lower=0 upper=1.6 effort=1 velocity=100 -> lower=0 upper=1.6698867696 effort=1 velocity=100; origin xyz=0.0028436 0.032651 -0.0003 rpy=0 0 0 -> xyz=0.0028436 0.032651 -0.0003 rpy=0 -0 0.0317598705691
- joint left_ring_1_joint: limit lower=0 upper=1.6 effort=1 velocity=100 -> lower=0 upper=1.60951229147 effort=1 velocity=100; origin xyz=-0.004945 0.11125 0.045939 rpy=1.5184 0 -1.5708 -> xyz=-0.004945 0.11125 0.045939 rpy=1.51838056831 -0.0272178525657 -1.56937222492
- joint left_ring_2_joint: limit lower=0 upper=1.6 effort=1 velocity=100 -> lower=0 upper=1.68998790605 effort=1 velocity=100; origin xyz=0.0031431 0.032624 -0.0003 rpy=0 0 0 -> xyz=0.0031431 0.032624 -0.0003 rpy=0 -0 0.0286180295277
- joint left_thumb_1_joint: limit lower=0 upper=0.92 effort=1 velocity=100 -> lower=0 upper=1.06242095936 effort=1 velocity=100; origin xyz=-0.0096402 -0.0097687 0.00125 rpy=1.5708 0 0.037536 -> xyz=-0.0096402 -0.0097687 0.00125 rpy=1.57080000191 0.0322660551661 0.037536118561
- joint left_thumb_2_joint: limit lower=0 upper=3.14 effort=1 velocity=100 -> lower=0 upper=0.424968383745 effort=1 velocity=100; origin xyz=-0.0385855343215257 0.0137354280979689 -0.00085000000007604 rpy=0 0 0 -> xyz=-0.0385855343215257 0.0137354280979689 -0.00085000000007604 rpy=0 0 -0.0129064220665
- joint left_thumb_3_joint: limit lower=0 upper=3.14 effort=1 velocity=100 -> lower=0 upper=0.637452575618 effort=1 velocity=100; origin xyz=-0.0204656980659991 0.00837680232935447 0.000199999999999881 rpy=0 0 0 -> xyz=-0.0204656980659991 0.00837680232935447 0.000199999999999881 rpy=0 0 -0.0193596330998
- joint left_thumb_swing_joint: limit lower=0 upper=1.70 effort=1 velocity=100 -> lower=0 upper=1.30899614247 effort=1 velocity=100; origin xyz=-0.035227 0.0908 -0.040206 rpy=0 0 0 -> xyz=-0.035227 0.0908 -0.040206 rpy=0 -0 0.224255962277
- joint right_index_1_joint: limit lower=0 upper=1.6 effort=1 velocity=100 -> lower=0 upper=1.60795403606 effort=1 velocity=100; origin xyz=-0.048156 -0.11125 0.045404 rpy=-1.6057 0 1.5708 -> xyz=-0.048156 -0.11125 0.045404 rpy=-1.60570928804 -0.0230624359379 1.57160543366
- joint right_index_2_joint: limit lower=0 upper=1.6 effort=1 velocity=100 -> lower=0 upper=1.68835173786 effort=1 velocity=100; origin xyz=0.00259487212105013 -0.0326721877470773 -0.000299999999999988 rpy=0 0 0 -> xyz=0.00259487212105013 -0.0326721877470773 -0.000299999999999988 rpy=0 -0 -0.0242303183457
- joint right_little_1_joint: limit lower=0 upper=1.6 effort=1 velocity=100 -> lower=0 upper=1.67172785459 effort=1 velocity=100; origin xyz=0.016446 -0.11125 0.042817 rpy=-1.4661 0 1.5708 -> xyz=0.016446 -0.11125 0.042817 rpy=-1.46609698912 -0.00756999419343 1.57000452558
- joint right_little_2_joint: limit lower=0 upper=1.6 effort=1 velocity=100 -> lower=0 upper=1.75531424732 effort=1 velocity=100; origin xyz=0.0023072 -0.032694 -0.0003 rpy=0 0 0 -> xyz=0.0023072 -0.032694 -0.0003 rpy=0 -0 -0.00799225759443
- joint right_middle_1_joint: limit lower=0 upper=1.6 effort=1 velocity=100 -> lower=0 upper=1.590368352 effort=1 velocity=100; origin xyz=-0.026577 -0.11125 0.046044 rpy=-1.5708 0 1.5708 -> xyz=-0.026577 -0.11125 0.046044 rpy=-1.57080000168 -0.0302474957799 1.57080011114
- joint right_middle_2_joint: limit lower=0 upper=1.6 effort=1 velocity=100 -> lower=0 upper=1.6698867696 effort=1 velocity=100; origin xyz=0.0028436 -0.032651 -0.0003 rpy=0 0 0 -> xyz=0.0028436 -0.032651 -0.0003 rpy=0 -0 -0.0317598705691
- joint right_ring_1_joint: limit lower=0 upper=1.6 effort=1 velocity=100 -> lower=0 upper=1.60951229147 effort=1 velocity=100; origin xyz=-0.004945 -0.11125 0.045939 rpy=-1.5184 0 1.5708 -> xyz=-0.004945 -0.11125 0.045939 rpy=-1.51838056831 -0.0272178525657 1.56937222492
- joint right_ring_2_joint: limit lower=0 upper=1.6 effort=1 velocity=100 -> lower=0 upper=1.68998790605 effort=1 velocity=100; origin xyz=0.0031431 -0.032624 -0.0003 rpy=0 0 0 -> xyz=0.0031431 -0.032624 -0.0003 rpy=0 -0 -0.0286180295277
- joint right_thumb_1_joint: limit lower=0 upper=0.92 effort=1 velocity=100 -> lower=0 upper=1.06242095936 effort=1 velocity=100; origin xyz=-0.0096402 0.0097687 0.00125 rpy=-1.5708 0 -0.037536 -> xyz=-0.0096402 0.0097687 0.00125 rpy=-1.57080000191 0.0322660551661 -0.037536118561
- joint right_thumb_2_joint: limit lower=0 upper=3.14 effort=1 velocity=100 -> lower=0 upper=0.424968383745 effort=1 velocity=100; origin xyz=-0.0385855343215257 -0.0137354280979689 -0.00085000000007604 rpy=0 0 0 -> xyz=-0.0385855343215257 -0.0137354280979689 -0.00085000000007604 rpy=0 0 0.0129064220665
- joint right_thumb_3_joint: limit lower=0 upper=3.14 effort=1 velocity=100 -> lower=0 upper=0.637452575618 effort=1 velocity=100; origin xyz=-0.0204656980659991 -0.00837680232935447 0.000199999999999881 rpy=0 0 0 -> xyz=-0.0204656980659991 -0.00837680232935447 0.000199999999999881 rpy=0 0 0.0193596330998
- joint right_thumb_swing_joint: limit lower=0 upper=1.70 effort=1 velocity=100 -> lower=0 upper=1.30899614247 effort=1 velocity=100; origin xyz=-0.035227 -0.0908 -0.040206 rpy=0 0 0 -> xyz=-0.035227 -0.0908 -0.040206 rpy=0 -0 -0.224255962277

File: ros_h1_2_ws/src/h1_2_inspire_description/urdf/h1_2_with_RH56DFTP_hands.urdf (robot description, URDF)
Before this commit: robot h1_2_with_RH56DFTP_hands, 58 links, 57 joints
Joints:
- joint left_index_1_joint: limit lower=0 upper=1.6 effort=1 velocity=100 -> lower=0 upper=1.60795403606 effort=1 velocity=100; origin xyz=-0.048156 0.11125 0.045404 rpy=1.6057 0 -1.5708 -> xyz=-0.048156 0.11125 0.045404 rpy=1.60570928804 -0.0230624359379 -1.57160543366
- joint left_index_2_joint: limit lower=0 upper=1.6 effort=1 velocity=100 -> lower=0 upper=1.68835173786 effort=1 velocity=100; origin xyz=0.00259487212105013 0.0326721877470773 -0.000299999999999988 rpy=0 0 0 -> xyz=0.00259487212105013 0.0326721877470773 -0.000299999999999988 rpy=0 -0 0.0242303183457
- joint left_little_1_joint: limit lower=0 upper=1.6 effort=1 velocity=100 -> lower=0 upper=1.67172785459 effort=1 velocity=100; origin xyz=0.016446 0.11125 0.042817 rpy=1.4661 0 -1.5708 -> xyz=0.016446 0.11125 0.042817 rpy=1.46609698912 -0.00756999419343 -1.57000452558
- joint left_little_2_joint: limit lower=0 upper=1.6 effort=1 velocity=100 -> lower=0 upper=1.75531424732 effort=1 velocity=100; origin xyz=0.0023072 0.032694 -0.0003 rpy=0 0 0 -> xyz=0.0023072 0.032694 -0.0003 rpy=0 -0 0.00799225759443
- joint left_middle_1_joint: limit lower=0 upper=1.6 effort=1 velocity=100 -> lower=0 upper=1.590368352 effort=1 velocity=100; origin xyz=-0.026577 0.11125 0.046044 rpy=1.5708 0 -1.5708 -> xyz=-0.026577 0.11125 0.046044 rpy=1.57080000168 -0.0302474957799 -1.57080011114
- joint left_middle_2_joint: limit lower=0 upper=1.6 effort=1 velocity=100 -> lower=0 upper=1.6698867696 effort=1 velocity=100; origin xyz=0.0028436 0.032651 -0.0003 rpy=0 0 0 -> xyz=0.0028436 0.032651 -0.0003 rpy=0 -0 0.0317598705691
- joint left_ring_1_joint: limit lower=0 upper=1.6 effort=1 velocity=100 -> lower=0 upper=1.60951229147 effort=1 velocity=100; origin xyz=-0.004945 0.11125 0.045939 rpy=1.5184 0 -1.5708 -> xyz=-0.004945 0.11125 0.045939 rpy=1.51838056831 -0.0272178525657 -1.56937222492
- joint left_ring_2_joint: limit lower=0 upper=1.6 effort=1 velocity=100 -> lower=0 upper=1.68998790605 effort=1 velocity=100; origin xyz=0.0031431 0.032624 -0.0003 rpy=0 0 0 -> xyz=0.0031431 0.032624 -0.0003 rpy=0 -0 0.0286180295277
- joint left_thumb_1_joint: limit lower=0 upper=0.92 effort=1 velocity=100 -> lower=0 upper=1.06242095936 effort=1 velocity=100; origin xyz=-0.0096402 -0.0097687 0.00125 rpy=1.5708 0 0.037536 -> xyz=-0.0096402 -0.0097687 0.00125 rpy=1.57080000191 0.0322660551661 0.037536118561
- joint left_thumb_2_joint: limit lower=0 upper=3.14 effort=1 velocity=100 -> lower=0 upper=0.424968383745 effort=1 velocity=100; origin xyz=-0.0385855343215257 0.0137354280979689 -0.00085000000007604 rpy=0 0 0 -> xyz=-0.0385855343215257 0.0137354280979689 -0.00085000000007604 rpy=0 0 -0.0129064220665
- joint left_thumb_3_joint: limit lower=0 upper=3.14 effort=1 velocity=100 -> lower=0 upper=0.637452575618 effort=1 velocity=100; origin xyz=-0.0204656980659991 0.00837680232935447 0.000199999999999881 rpy=0 0 0 -> xyz=-0.0204656980659991 0.00837680232935447 0.000199999999999881 rpy=0 0 -0.0193596330998
- joint left_thumb_swing_joint: limit lower=0 upper=1.70 effort=1 velocity=100 -> lower=0 upper=1.30899614247 effort=1 velocity=100; origin xyz=-0.035227 0.0908 -0.040206 rpy=0 0 0 -> xyz=-0.035227 0.0908 -0.040206 rpy=0 -0 0.224255962277
- joint right_index_1_joint: limit lower=0 upper=1.6 effort=1 velocity=100 -> lower=0 upper=1.60795403606 effort=1 velocity=100; origin xyz=-0.048156 -0.11125 0.045404 rpy=-1.6057 0 1.5708 -> xyz=-0.048156 -0.11125 0.045404 rpy=-1.60570928804 -0.0230624359379 1.57160543366
- joint right_index_2_joint: limit lower=0 upper=1.6 effort=1 velocity=100 -> lower=0 upper=1.68835173786 effort=1 velocity=100; origin xyz=0.00259487212105013 -0.0326721877470773 -0.000299999999999988 rpy=0 0 0 -> xyz=0.00259487212105013 -0.0326721877470773 -0.000299999999999988 rpy=0 -0 -0.0242303183457
- joint right_little_1_joint: limit lower=0 upper=1.6 effort=1 velocity=100 -> lower=0 upper=1.67172785459 effort=1 velocity=100; origin xyz=0.016446 -0.11125 0.042817 rpy=-1.4661 0 1.5708 -> xyz=0.016446 -0.11125 0.042817 rpy=-1.46609698912 -0.00756999419343 1.57000452558
- joint right_little_2_joint: limit lower=0 upper=1.6 effort=1 velocity=100 -> lower=0 upper=1.75531424732 effort=1 velocity=100; origin xyz=0.0023072 -0.032694 -0.0003 rpy=0 0 0 -> xyz=0.0023072 -0.032694 -0.0003 rpy=0 -0 -0.00799225759443
- joint right_middle_1_joint: limit lower=0 upper=1.6 effort=1 velocity=100 -> lower=0 upper=1.590368352 effort=1 velocity=100; origin xyz=-0.026577 -0.11125 0.046044 rpy=-1.5708 0 1.5708 -> xyz=-0.026577 -0.11125 0.046044 rpy=-1.57080000168 -0.0302474957799 1.57080011114
- joint right_middle_2_joint: limit lower=0 upper=1.6 effort=1 velocity=100 -> lower=0 upper=1.6698867696 effort=1 velocity=100; origin xyz=0.0028436 -0.032651 -0.0003 rpy=0 0 0 -> xyz=0.0028436 -0.032651 -0.0003 rpy=0 -0 -0.0317598705691
- joint right_ring_1_joint: limit lower=0 upper=1.6 effort=1 velocity=100 -> lower=0 upper=1.60951229147 effort=1 velocity=100; origin xyz=-0.004945 -0.11125 0.045939 rpy=-1.5184 0 1.5708 -> xyz=-0.004945 -0.11125 0.045939 rpy=-1.51838056831 -0.0272178525657 1.56937222492
- joint right_ring_2_joint: limit lower=0 upper=1.6 effort=1 velocity=100 -> lower=0 upper=1.68998790605 effort=1 velocity=100; origin xyz=0.0031431 -0.032624 -0.0003 rpy=0 0 0 -> xyz=0.0031431 -0.032624 -0.0003 rpy=0 -0 -0.0286180295277
- joint right_thumb_1_joint: limit lower=0 upper=0.92 effort=1 velocity=100 -> lower=0 upper=1.06242095936 effort=1 velocity=100; origin xyz=-0.0096402 0.0097687 0.00125 rpy=-1.5708 0 -0.037536 -> xyz=-0.0096402 0.0097687 0.00125 rpy=-1.57080000191 0.0322660551661 -0.037536118561
- joint right_thumb_2_joint: limit lower=0 upper=3.14 effort=1 velocity=100 -> lower=0 upper=0.424968383745 effort=1 velocity=100; origin xyz=-0.0385855343215257 -0.0137354280979689 -0.00085000000007604 rpy=0 0 0 -> xyz=-0.0385855343215257 -0.0137354280979689 -0.00085000000007604 rpy=0 0 0.0129064220665
- joint right_thumb_3_joint: limit lower=0 upper=3.14 effort=1 velocity=100 -> lower=0 upper=0.637452575618 effort=1 velocity=100; origin xyz=-0.0204656980659991 -0.00837680232935447 0.000199999999999881 rpy=0 0 0 -> xyz=-0.0204656980659991 -0.00837680232935447 0.000199999999999881 rpy=0 0 0.0193596330998
- joint right_thumb_swing_joint: limit lower=0 upper=1.70 effort=1 velocity=100 -> lower=0 upper=1.30899614247 effort=1 velocity=100; origin xyz=-0.035227 -0.0908 -0.040206 rpy=0 0 0 -> xyz=-0.035227 -0.0908 -0.040206 rpy=0 -0 -0.224255962277
