Commit message: Manos: q=0 es la mano abierta y el limite superior la mano cerrada
Los ceros y limites de las 12 juntas de cada mano se fijan ahora desde el
manual de usuario de la RH56DFTP, apartado 2.6.11 (paginas impresas 21 y 22),
que define un angulo de cuerda por DOF contra el plano metacarpiano:

  dedos            alpha   176 (abierto) -> 20 (cerrado)
  pulgar flexion   theta    70           -> -13
  pulgar rotacion  beta    165           -> 90

No son angulos articulares, asi que se calcularon sobre el modelo y se
resolvio que valor de q produce cada extremo. Cada origen de junta se giro
para que q=0 caiga exactamente en el angulo de abierto, y el limite superior
en el de cerrado:

  junta          giro del cero     q_max (rad)
  index_1          -1.32 deg        1.60795
  middle_1         -1.73 deg        1.59037
  ring_1           -1.56 deg        1.60951
  little_1         -0.44 deg        1.67173
  thumb_1          +1.85 deg        1.06242
  thumb_swing     +12.85 deg        1.30900

Las cuatro q_max de los dedos difieren porque cada dedo asienta en la palma
con su propio angulo, de modo que el mismo barrido 176..20 cuesta un recorrido
articular algo distinto. Las mimic llevan multiplicador * q_max y su cero se
giro multiplicador * delta, o la falange distal no quedaria en su sitio con
q=0.

Ningun eje cambia: los seis cierran al crecer q. Con eso el mapeo al SDK es
uno solo para los seis:

  ANGLE_SET = 1000 * (1 - q / q_max)

Dos correcciones de camino, ambas detectadas al contrastar con el modelo:

- Una medida intermedia tomaba beta como angulo 3D contra la normal de la
  palma, cuando la figura del manual es una vista superior y hay que proyectar
  al plano x-y. Esa medida hacia creer que el swing del pulgar corria invertido
  respecto a los otros cinco DOF y que habia que voltear su eje. No es asi:
  beta decrece con q como los demas. El usuario lo detecto en RViz, donde
  swing=1.5331 se ve como beta~90 y swing=0 como beta~180, que es justo lo que
  da la definicion correcta (90.0 y 177.8).
- El primer calculo de los limites superiores tomaba la yema como el vertice
  mas lejano en cada configuracion, que cambia al curvarse el dedo, en vez de
  un punto material fijo. Daba extremos pasados de 3.5 a 5 grados.

Verificacion:
  los 12 extremos sobre el modelo    error maximo 4.6e-05 grados
  simetria izq/der, misma consigna   0.000000 mm en abierta, cerrada y 2 aleatorias
  autocolision al cierre total       los 4 dedos ya no tocan la palma (antes el
                                     medio penetraba 0.51 mm); solo el pulgar
                                     apoya, 2.78 mm contra la palma y 0.37 mm
                                     contra el indice
  XML 9/9, xacro 3/3, check_urdf 6/6, nq=46 nv=45, masa 68.6640 kg

Comprobado ademas visualmente en RViz con display_h1_2_with_hands.launch.py:
a q=0 los cuatro dedos quedan casi rectos y el pulgar abierto, y a q_max la
mano cierra en puno con el pulgar encima.

Se propagan el espejo a la mano derecha y los dos URDF planos; h1_2_handless
no se toca porque no lleva manos.

Co-Authored-By: Claude Opus 5 <noreply@anthropic.com>
Claude-Session: https://claude.ai/code/session_01WDAX8VZbrLhjdUkohUZLGo

File: ros_h1_2_ws/src/h1_2_inspire_description/urdf/inspire_hand_left.urdf.xacro (robot description, xacro)
@@ -15,5 +15,23 @@
      NOT in the visual or collision model. The centre of mass is unchanged and
      the tensor is scaled by 0.696619/0.314091 = 2.217891, which keeps the
-     vendor's mass distribution. Both palms carry the same values, mirrored. -->
+     vendor's mass distribution. Both palms carry the same values, mirrored.
+     Joint zeros and limits follow the RH56DFTP user manual, section 2.6.11
+     (printed pages 21 and 22), which defines one chord angle per DOF against
+     the metacarpal plane. For every actuated joint q=0 is the hand FULLY OPEN
+     and the upper limit is FULLY CLOSED, so the SDK scale maps uniformly:
+       ANGLE_SET = 1000 * (1 - q / q_max)        q = q_max * (1 - ANGLE_SET/1000)
+     | DOF            | manual angle    | open  | closed | q_max (rad) |
+     | fingers        | alpha           | 176   | 20     | see below   |
+     | thumb bending  | theta           | 70    | -13    | 1.06242     |
+     | thumb rotation | beta            | 165   | 90     | 1.30900     |
+     q_max per finger: index 1.60795, middle 1.59037, ring 1.60951,
+     little 1.67173. They differ because each finger seats at its own angle on
+     the palm, so the same 176..20 sweep needs a slightly different joint
+     travel. The mimic joints carry multiplier * q_max.
+     Every joint origin was rotated so that q=0 lands exactly on the open
+     angle; the shifts were 0.4 to 1.9 degrees except thumb_swing, which moved
+     12.85 degrees. No joint axis was changed: all six close as q grows.
+     Verified by computing the manual's angles on this model: all twelve
+     endpoints land on target to better than 0.001 degrees. -->
 <robot xmlns:xacro="http://www.ros.org/wiki/xacro">
   <link name="left_hand_base_link">
@@ -64,9 +82,9 @@
   </link>
   <joint name="left_thumb_swing_joint" type="revolute">
-    <origin xyz="-0.035227 0.0908 -0.040206" rpy="0 0 0"/>
+    <origin xyz="-0.035227 0.0908 -0.040206" rpy="0 -0 0.224255962277"/>
     <parent link="left_hand_base_link"/>
     <child link="left_thumb_swing"/>
     <axis xyz="0 0 1"/>
-    <limit lower="0" upper="1.70" effort="1" velocity="100"/>
+    <limit lower="0" upper="1.30899614247" effort="1" velocity="100"/>
   </joint>
   <link name="left_thumb_1">
@@ -94,9 +112,9 @@
   </link>
   <joint name="left_thumb_1_joint" type="revolute">
-    <origin xyz="-0.0096402 -0.0097687 0.00125" rpy="1.5708 0 0.037536"/>
+    <origin xyz="-0.0096402 -0.0097687 0.00125" rpy="1.57080000191 0.0322660551661 0.037536118561"/>
     <parent link="left_thumb_swing"/>
     <child link="left_thumb_1"/>
     <axis xyz="0 0 -1"/>
-    <limit lower="0" upper="0.92" effort="1" velocity="100"/>
+    <limit lower="0" upper="1.06242095936" effort="1" velocity="100"/>
   </joint>
   <link name="left_thumb_2">
@@ -124,9 +142,9 @@
   </link>
   <joint name="left_thumb_2_joint" type="revolute">
-    <origin xyz="-0.0385855343215257 0.0137354280979689 -0.00085000000007604" rpy="0 0 0"/>
+    <origin xyz="-0.0385855343215257 0.0137354280979689 -0.00085000000007604" rpy="0 0 -0.0129064220665"/>
     <parent link="left_thumb_1"/>
     <child link="left_thumb_2"/>
     <axis xyz="0 0 -1"/>
-    <limit lower="0" upper="3.14" effort="1" velocity="100"/>
+    <limit lower="0" upper="0.424968383745" effort="1" velocity="100"/>
     <mimic joint="left_thumb_1_joint" multiplier="0.40" offset="0"/>
   </joint>
@@ -155,9 +173,9 @@
   </link>
   <joint name="left_thumb_3_joint" type="revolute">
-    <origin xyz="-0.0204656980659991 0.00837680232935447 0.000199999999999881" rpy="0 0 0"/>
+    <origin xyz="-0.0204656980659991 0.00837680232935447 0.000199999999999881" rpy="0 0 -0.0193596330998"/>
     <parent link="left_thumb_2"/>
     <child link="left_thumb_3"/>
     <axis xyz="0 0 -1"/>
-    <limit lower="0" upper="3.14" effort="1" velocity="100"/>
+    <limit lower="0" upper="0.637452575618" effort="1" velocity="100"/>
     <mimic joint="left_thumb_1_joint" multiplier="0.60" offset="0"/>
   </joint>
@@ -186,9 +204,9 @@
   </link>
   <joint name="left_index_1_joint" type="revolute">
-    <origin xyz="-0.048156 0.11125 0.045404" rpy="1.6057 0 -1.5708"/>
+    <origin xyz="-0.048156 0.11125 0.045404" rpy="1.60570928804 -0.0230624359379 -1.57160543366"/>
     <parent link="left_hand_base_link"/>
     <child link="left_index_1"/>
     <axis xyz="0 0 -1"/>
-    <limit lower="0" upper="1.6" effort="1" velocity="100"/>
+    <limit lower="0" upper="1.60795403606" effort="1" velocity="100"/>
   </joint>
   <link name="left_index_2">
@@ -216,9 +234,9 @@
   </link>
   <joint name="left_index_2_joint" type="revolute">
-    <origin xyz="0.00259487212105013 0.0326721877470773 -0.000299999999999988" rpy="0 0 0"/>
+    <origin xyz="0.00259487212105013 0.0326721877470773 -0.000299999999999988" rpy="0 -0 0.0242303183457"/>
     <parent link="left_index_1"/>
     <child link="left_index_2"/>
     <axis xyz="0 0 -1"/>
-    <limit lower="0" upper="1.6" effort="1" velocity="100"/>
+    <limit lower="0" upper="1.68835173786" effort="1" velocity="100"/>
     <mimic joint="left_index_1_joint" multiplier="1.05" offset="0"/>
   </joint>
@@ -247,9 +265,9 @@
   </link>
   <joint name="left_middle_1_joint" type="revolute">
-    <origin xyz="-0.026577 0.11125 0.046044" rpy="1.5708 0 -1.5708"/>
+    <origin xyz="-0.026577 0.11125 0.046044" rpy="1.57080000168 -0.0302474957799 -1.57080011114"/>
     <parent link="left_hand_base_link"/>
     <child link="left_middle_1"/>
     <axis xyz="0 0 -1"/>
-    <limit lower="0" upper="1.6" effort="1" velocity="100"/>
+    <limit lower="0" upper="1.590368352" effort="1" velocity="100"/>
   </joint>
   <link name="left_middle_2">
@@ -277,9 +295,9 @@
   </link>
   <joint name="left_middle_2_joint" type="revolute">
-    <origin xyz="0.0028436 0.032651 -0.0003" rpy="0 0 0"/>
+    <origin xyz="0.0028436 0.032651 -0.0003" rpy="0 -0 0.0317598705691"/>
     <parent link="left_middle_1"/>
     <child link="left_middle_2"/>
     <axis xyz="0 0 -1"/>
-    <limit lower="0" upper="1.6" effort="1" velocity="100"/>
+    <limit lower="0" upper="1.6698867696" effort="1" velocity="100"/>
     <mimic joint="left_middle_1_joint" multiplier="1.05" offset="0"/>
   </joint>
@@ -308,9 +326,9 @@
   </link>
   <joint name="left_ring_1_joint" type="revolute">
-    <origin xyz="-0.004945 0.11125 0.045939" rpy="1.5184 0 -1.5708"/>
+    <origin xyz="-0.004945 0.11125 0.045939" rpy="1.51838056831 -0.0272178525657 -1.56937222492"/>
     <parent link="left_hand_base_link"/>
     <child link="left_ring_1"/>
     <axis xyz="0 0 -1"/>
-    <limit lower="0" upper="1.6" effort="1" velocity="100"/>
+    <limit lower="0" upper="1.60951229147" effort="1" velocity="100"/>
   </joint>
   <link name="left_ring_2">
@@ -338,9 +356,9 @@
   </link>
   <joint name="left_ring_2_joint" type="revolute">
-    <origin xyz="0.0031431 0.032624 -0.0003" rpy="0 0 0"/>
+    <origin xyz="0.0031431 0.032624 -0.0003" rpy="0 -0 0.0286180295277"/>
     <parent link="left_ring_1"/>
     <child link="left_ring_2"/>
     <axis xyz="0 0 -1"/>
-    <limit lower="0" upper="1.6" effort="1" velocity="100"/>
+    <limit lower="0" upper="1.68998790605" effort="1" velocity="100"/>
     <mimic joint="left_ring_1_joint" multiplier="1.05" offset="0"/>
   </joint>
@@ -369,9 +387,9 @@
   </link>
   <joint name="left_little_1_joint" type="revolute">
-    <origin xyz="0.016446 0.11125 0.042817" rpy="1.4661 0 -1.5708"/>
+    <origin xyz="0.016446 0.11125 0.042817" rpy="1.46609698912 -0.00756999419343 -1.57000452558"/>
     <parent link="left_hand_base_link"/>
     <child link="left_little_1"/>
     <axis xyz="0 0 -1"/>
-    <limit lower="0" upper="1.6" effort="1" velocity="100"/>
+    <limit lower="0" upper="1.67172785459" effort="1" velocity="100"/>
   </joint>
   <link name="left_little_2">
@@ -399,9 +417,9 @@
   </link>
   <joint name="left_little_2_joint" type="revolute">
-    <origin xyz="0.0023072 0.032694 -0.0003" rpy="0 0 0"/>
+    <origin xyz="0.0023072 0.032694 -0.0003" rpy="0 -0 0.00799225759443"/>
     <parent link="left_little_1"/>
     <child link="left_little_2"/>
     <axis xyz="0 0 -1"/>
-    <limit lower="0" upper="1.6" effort="1" velocity="100"/>
+    <limit lower="0" upper="1.75531424732" effort="1" velocity="100"/>
     <mimic joint="left_little_1_joint" multiplier="1.05" offset="0"/>
   </joint>

File: ros_h1_2_ws/src/h1_2_inspire_description/urdf/inspire_hand_right.urdf.xacro (robot description, xacro)
@@ -22,5 +22,23 @@
      NOT in the visual or collision model. The centre of mass is unchanged and
      the tensor is scaled by 0.696619/0.314091 = 2.217891, which keeps the
-     vendor's mass distribution. Both palms carry the same values, mirrored. -->
+     vendor's mass distribution. Both palms carry the same values, mirrored.
+     Joint zeros and limits follow the RH56DFTP user manual, section 2.6.11
+     (printed pages 21 and 22), which defines one chord angle per DOF against
+     the metacarpal plane. For every actuated joint q=0 is the hand FULLY OPEN
+     and the upper limit is FULLY CLOSED, so the SDK scale maps uniformly:
+       ANGLE_SET = 1000 * (1 - q / q_max)        q = q_max * (1 - ANGLE_SET/1000)
+     | DOF            | manual angle    | open  | closed | q_max (rad) |
+     | fingers        | alpha           | 176   | 20     | see below   |
+     | thumb bending  | theta           | 70    | -13    | 1.06242     |
+     | thumb rotation | beta            | 165   | 90     | 1.30900     |
+     q_max per finger: index 1.60795, middle 1.59037, ring 1.60951,
+     little 1.67173. They differ because each finger seats at its own angle on
+     the palm, so the same 176..20 sweep needs a slightly different joint
+     travel. The mimic joints carry multiplier * q_max.
+     Every joint origin was rotated so that q=0 lands exactly on the open
+     angle; the shifts were 0.4 to 1.9 degrees except thumb_swing, which moved
+     12.85 degrees. No joint axis was changed: all six close as q grows.
+     Verified by computing the manual's angles on this model: all twelve
+     endpoints land on target to better than 0.001 degrees. -->
 <robot xmlns:xacro="http://www.ros.org/wiki/xacro">
   <link name="right_hand_base_link">
@@ -71,9 +89,9 @@
   </link>
   <joint name="right_thumb_swing_joint" type="revolute">
-    <origin xyz="-0.035227 -0.0908 -0.040206" rpy="0 0 0"/>
+    <origin xyz="-0.035227 -0.0908 -0.040206" rpy="0 -0 -0.224255962277"/>
     <parent link="right_hand_base_link"/>
     <child link="right_thumb_swing"/>
     <axis xyz="0 0 -1"/>
-    <limit lower="0" upper="1.70" effort="1" velocity="100"/>
+    <limit lower="0" upper="1.30899614247" effort="1" velocity="100"/>
   </joint>
   <link name="right_thumb_1">
@@ -101,9 +119,9 @@
   </link>
   <joint name="right_thumb_1_joint" type="revolute">
-    <origin xyz="-0.0096402 0.0097687 0.00125" rpy="-1.5708 0 -0.037536"/>
+    <origin xyz="-0.0096402 0.0097687 0.00125" rpy="-1.57080000191 0.0322660551661 -0.037536118561"/>
     <parent link="right_thumb_swing"/>
     <child link="right_thumb_1"/>
     <axis xyz="0 0 1"/>
-    <limit lower="0" upper="0.92" effort="1" velocity="100"/>
+    <limit lower="0" upper="1.06242095936" effort="1" velocity="100"/>
   </joint>
   <link name="right_thumb_2">
@@ -131,9 +149,9 @@
   </link>
   <joint name="right_thumb_2_joint" type="revolute">
-    <origin xyz="-0.0385855343215257 -0.0137354280979689 -0.00085000000007604" rpy="0 0 0"/>
+    <origin xyz="-0.0385855343215257 -0.0137354280979689 -0.00085000000007604" rpy="0 0 0.0129064220665"/>
     <parent link="right_thumb_1"/>
     <child link="right_thumb_2"/>
     <axis xyz="0 0 1"/>
-    <limit lower="0" upper="3.14" effort="1" velocity="100"/>
+    <limit lower="0" upper="0.424968383745" effort="1" velocity="100"/>
     <mimic joint="right_thumb_1_joint" multiplier="0.40" offset="0"/>
   </joint>
@@ -162,9 +180,9 @@
   </link>
   <joint name="right_thumb_3_joint" type="revolute">
-    <origin xyz="-0.0204656980659991 -0.00837680232935447 0.000199999999999881" rpy="0 0 0"/>
+    <origin xyz="-0.0204656980659991 -0.00837680232935447 0.000199999999999881" rpy="0 0 0.0193596330998"/>
     <parent link="right_thumb_2"/>
     <child link="right_thumb_3"/>
     <axis xyz="0 0 1"/>
-    <limit lower="0" upper="3.14" effort="1" velocity="100"/>
+    <limit lower="0" upper="0.637452575618" effort="1" velocity="100"/>
     <mimic joint="right_thumb_1_joint" multiplier="0.60" offset="0"/>
   </joint>
@@ -193,9 +211,9 @@
   </link>
   <joint name="right_index_1_joint" type="revolute">
-    <origin xyz="-0.048156 -0.11125 0.045404" rpy="-1.6057 0 1.5708"/>
+    <origin xyz="-0.048156 -0.11125 0.045404" rpy="-1.60570928804 -0.0230624359379 1.57160543366"/>
     <parent link="right_hand_base_link"/>
     <child link="right_index_1"/>
     <axis xyz="0 0 1"/>
-    <limit lower="0" upper="1.6" effort="1" velocity="100"/>
+    <limit lower="0" upper="1.60795403606" effort="1" velocity="100"/>
   </joint>
   <link name="right_index_2">
@@ -223,9 +241,9 @@
   </link>
   <joint name="right_index_2_joint" type="revolute">
-    <origin xyz="0.00259487212105013 -0.0326721877470773 -0.000299999999999988" rpy="0 0 0"/>
+    <origin xyz="0.00259487212105013 -0.0326721877470773 -0.000299999999999988" rpy="0 -0 -0.0242303183457"/>
     <parent link="right_index_1"/>
     <child link="right_index_2"/>
     <axis xyz="0 0 1"/>
-    <limit lower="0" upper="1.6" effort="1" velocity="100"/>
+    <limit lower="0" upper="1.68835173786" effort="1" velocity="100"/>
     <mimic joint="right_index_1_joint" multiplier="1.05" offset="0"/>
   </joint>
@@ -254,9 +272,9 @@
   </link>
   <joint name="right_middle_1_joint" type="revolute">
-    <origin xyz="-0.026577 -0.11125 0.046044" rpy="-1.5708 0 1.5708"/>
+    <origin xyz="-0.026577 -0.11125 0.046044" rpy="-1.57080000168 -0.0302474957799 1.57080011114"/>
     <parent link="right_hand_base_link"/>
     <child link="right_middle_1"/>
     <axis xyz="0 0 1"/>
-    <limit lower="0" upper="1.6" effort="1" velocity="100"/>
+    <limit lower="0" upper="1.590368352" effort="1" velocity="100"/>
   </joint>
   <link name="right_middle_2">
@@ -284,9 +302,9 @@
   </link>
   <joint name="right_middle_2_joint" type="revolute">
-    <origin xyz="0.0028436 -0.032651 -0.0003" rpy="0 0 0"/>
+    <origin xyz="0.0028436 -0.032651 -0.0003" rpy="0 -0 -0.0317598705691"/>
     <parent link="right_middle_1"/>
     <child link="right_middle_2"/>
     <axis xyz="0 0 1"/>
-    <limit lower="0" upper="1.6" effort="1" velocity="100"/>
+    <limit lower="0" upper="1.6698867696" effort="1" velocity="100"/>
     <mimic joint="right_middle_1_joint" multiplier="1.05" offset="0"/>
   </joint>
@@ -315,9 +333,9 @@
   </link>
   <joint name="right_ring_1_joint" type="revolute">
-    <origin xyz="-0.004945 -0.11125 0.045939" rpy="-1.5184 0 1.5708"/>
+    <origin xyz="-0.004945 -0.11125 0.045939" rpy="-1.51838056831 -0.0272178525657 1.56937222492"/>
     <parent link="right_hand_base_link"/>
     <child link="right_ring_1"/>
     <axis xyz="0 0 1"/>
-    <limit lower="0" upper="1.6" effort="1" velocity="100"/>
+    <limit lower="0" upper="1.60951229147" effort="1" velocity="100"/>
   </joint>
   <link name="right_ring_2">
@@ -345,9 +363,9 @@
   </link>
   <joint name="right_ring_2_joint" type="revolute">
-    <origin xyz="0.0031431 -0.032624 -0.0003" rpy="0 0 0"/>
+    <origin xyz="0.0031431 -0.032624 -0.0003" rpy="0 -0 -0.0286180295277"/>
     <parent link="right_ring_1"/>
     <child link="right_ring_2"/>
     <axis xyz="0 0 1"/>
-    <limit lower="0" upper="1.6" effort="1" velocity="100"/>
+    <limit lower="0" upper="1.68998790605" effort="1" velocity="100"/>
     <mimic joint="right_ring_1_joint" multiplier="1.05" offset="0"/>
   </joint>
@@ -376,9 +394,9 @@
   </link>
   <joint name="right_little_1_joint" type="revolute">
-    <origin xyz="0.016446 -0.11125 0.042817" rpy="-1.4661 0 1.5708"/>
+    <origin xyz="0.016446 -0.11125 0.042817" rpy="-1.46609698912 -0.00756999419343 1.57000452558"/>
     <parent link="right_hand_base_link"/>
     <child link="right_little_1"/>
     <axis xyz="0 0 1"/>
-    <limit lower="0" upper="1.6" effort="1" velocity="100"/>
+    <limit lower="0" upper="1.67172785459" effort="1" velocity="100"/>
   </joint>
   <link name="right_little_2">
@@ -406,9 +424,9 @@
   </link>
   <joint name="right_little_2_joint" type="revolute">
-    <origin xyz="0.0023072 -0.032694 -0.0003" rpy="0 0 0"/>
+    <origin xyz="0.0023072 -0.032694 -0.0003" rpy="0 -0 -0.00799225759443"/>
     <parent link="right_little_1"/>
     <child link="right_little_2"/>
     <axis xyz="0 0 1"/>
-    <limit lower="0" upper="1.6" effort="1" velocity="100"/>
+    <limit lower="0" upper="1.75531424732" effort="1" velocity="100"/>
     <mimic joint="right_little_1_joint" multiplier="1.05" offset="0"/>
   </joint>
