Commit message: Manos: limites superiores y acoplamiento medidos sobre la mano real
Los limites de cierre del commit 074de3e salian de los angulos nominales del
manual, y la mano real no llega a ellos: en RViz los dedos cerraban contra la
palma y, con el swing y la flexion del pulgar al maximo, la punta del pulgar
atravesaba la palma. Ahora salen de fotos de la mano real a ANGLE_SET = 0, 500
y 1000 (inspire_hand_interface/Caracterizacion/imagenes/angulos limite).

Metodo: el modelo se renderiza en MuJoCo con una camara virtual ajustada a cada
foto con las partes que no se mueven (palma y dedos abiertos), y se barren los
valores articulares hasta que la silueta renderizada coincide con la
fotografiada. Para las fotos de la rotacion del pulgar, que miran a lo largo
del eje del swing, la camara es de 6 GDL, se inicializa por PnP con 8 puntos
de los dedos y se refina con las siluetas.

Cambios, en las dos manos (la derecha regenerada por espejo):

  *_index/middle/ring/little_1   1.59..1.67 -> 1.620 (comun a los cuatro)
  *_*_2 (mimic)                  x1.05      -> x0.85, upper 1.377
  *_thumb_1                      1.0624     -> 0.660
  *_thumb_2 / *_thumb_3          upper 0.264 / 0.396 (x0.40 / x0.60 sin cambio)
  *_thumb_swing                  1.309      -> 1.190

Los ceros no cambian: siguen el manual (alpha 176, theta 70, beta 165) y las
fotos de la mano abierta los confirman a unos 3 grados (3 a 6 en la rotacion
del pulgar).

Lo que dicen las fotos:
- Al cierre real los dedos quedan en alpha 31..37 (manual 20), la flexion del
  pulgar en theta ~19 (manual -13) y la rotacion en beta 96..97 (manual 90).
- La proximal de los dedos ya estaba casi bien; lo que fallaba era el
  multiplicador 1.05, que doblaba la distal hacia la palma. Las cuatro fotos
  piden un q1 de 1.58 a 1.74; 1.620 con x0.85 es el par comun de menor error
  conjunto.
- El acoplamiento real no es lineal (q2/q1 ~0.65 a mitad de recorrido, 0.82
  al cierre). Como una mimic de URDF solo puede ser lineal, 0.85 reproduce el
  cierre a 0.5 grados de orientacion de la yema y deja la yema unos 13 grados
  demasiado doblada a ANGLE_SET = 500.
- El mapeo del SDK no es lineal en la proximal: a ANGLE_SET = 500 los dedos ya
  llevan el 64 % del recorrido. El README sustituye la formula lineal por una
  tabla de interpolacion (0 / 1.05 / 1.620 para los dedos, 0 / 0.38 / 0.660
  para thumb_1) con funciones angle_set_to_q / q_to_angle_set.
- Los multiplicadores del pulgar 0.40 / 0.60 no se pueden resolver con estas
  fotos y quedan como estaban.

Verificacion:
  IoU con la foto, region del digito cerrado, valores leidos de los archivos
    indice 0.725 -> 0.868   medio 0.714 -> 0.849   anular 0.737 -> 0.817
    menique 0.777 -> 0.859  pulgar 0.481 -> 0.799
  swing max + bend max: punta del pulgar a 33.1 mm de la palma (antes la
    atravesaba); todo cerrado: dedos a 12..18 mm de la palma
  mimic=True en Pinocchio aplica 0.85 (0.0000 grados de error)
  simetria izq/der 0.000000 mm; XML 9/9; xacro + check_urdf 7/7;
    nq=46 nv=45; 68.6640 kg; plano identico al xacro
  comprobado ademas visualmente en RViz por el usuario

Se actualizan las cabeceras de ambos xacro, el README (seccion de manos y
tabla de acoplamiento de Isaac) y los URDF planos h1_2_with_RH56DFTP_hands y
h1_2_hands_isaac.

Co-Authored-By: Claude Opus 5.5 <noreply@anthropic.com>
Claude-Session: https://claude.ai/code/session_01WDAX8VZbrLhjdUkohUZLGo

File: ros_h1_2_ws/src/h1_2_inspire_description/urdf/h1_2_hands_isaac.urdf (robot description, URDF)
Before this commit: robot h1_2_with_inspire_hands, 58 links, 57 joints
Joints:
- joint left_index_1_joint: limit lower=0 upper=1.60795403606 effort=1 velocity=100 -> lower=0 upper=1.62 effort=1 velocity=100
- joint left_index_2_joint: limit lower=0 upper=1.68835173786 effort=1 velocity=100 -> lower=0 upper=1.377 effort=1 velocity=100
- joint left_little_1_joint: limit lower=0 upper=1.67172785459 effort=1 velocity=100 -> lower=0 upper=1.62 effort=1 velocity=100
- joint left_little_2_joint: limit lower=0 upper=1.75531424732 effort=1 velocity=100 -> lower=0 upper=1.377 effort=1 velocity=100
- joint left_middle_1_joint: limit lower=0 upper=1.590368352 effort=1 velocity=100 -> lower=0 upper=1.62 effort=1 velocity=100
- joint left_middle_2_joint: limit lower=0 upper=1.6698867696 effort=1 velocity=100 -> lower=0 upper=1.377 effort=1 velocity=100
- joint left_ring_1_joint: limit lower=0 upper=1.60951229147 effort=1 velocity=100 -> lower=0 upper=1.62 effort=1 velocity=100
- joint left_ring_2_joint: limit lower=0 upper=1.68998790605 effort=1 velocity=100 -> lower=0 upper=1.377 effort=1 velocity=100
- joint left_thumb_1_joint: limit lower=0 upper=1.06242095936 effort=1 velocity=100 -> lower=0 upper=0.66 effort=1 velocity=100
- joint left_thumb_2_joint: limit lower=0 upper=0.424968383745 effort=1 velocity=100 -> lower=0 upper=0.264 effort=1 velocity=100
- joint left_thumb_3_joint: limit lower=0 upper=0.637452575618 effort=1 velocity=100 -> lower=0 upper=0.396 effort=1 velocity=100
- joint left_thumb_swing_joint: limit lower=0 upper=1.30899614247 effort=1 velocity=100 -> lower=0 upper=1.19 effort=1 velocity=100
- joint right_index_1_joint: limit lower=0 upper=1.60795403606 effort=1 velocity=100 -> lower=0 upper=1.62 effort=1 velocity=100
- joint right_index_2_joint: limit lower=0 upper=1.68835173786 effort=1 velocity=100 -> lower=0 upper=1.377 effort=1 velocity=100
- joint right_little_1_joint: limit lower=0 upper=1.67172785459 effort=1 velocity=100 -> lower=0 upper=1.62 effort=1 velocity=100
- joint right_little_2_joint: limit lower=0 upper=1.75531424732 effort=1 velocity=100 -> lower=0 upper=1.377 effort=1 velocity=100
- joint right_middle_1_joint: limit lower=0 upper=1.590368352 effort=1 velocity=100 -> lower=0 upper=1.62 effort=1 velocity=100
- joint right_middle_2_joint: limit lower=0 upper=1.6698867696 effort=1 velocity=100 -> lower=0 upper=1.377 effort=1 velocity=100
- joint right_ring_1_joint: limit lower=0 upper=1.60951229147 effort=1 velocity=100 -> lower=0 upper=1.62 effort=1 velocity=100
- joint right_ring_2_joint: limit lower=0 upper=1.68998790605 effort=1 velocity=100 -> lower=0 upper=1.377 effort=1 velocity=100
- joint right_thumb_1_joint: limit lower=0 upper=1.06242095936 effort=1 velocity=100 -> lower=0 upper=0.66 effort=1 velocity=100
- joint right_thumb_2_joint: limit lower=0 upper=0.424968383745 effort=1 velocity=100 -> lower=0 upper=0.264 effort=1 velocity=100
- joint right_thumb_3_joint: limit lower=0 upper=0.637452575618 effort=1 velocity=100 -> lower=0 upper=0.396 effort=1 velocity=100
- joint right_thumb_swing_joint: limit lower=0 upper=1.30899614247 effort=1 velocity=100 -> lower=0 upper=1.19 effort=1 velocity=100

File: ros_h1_2_ws/src/h1_2_inspire_description/urdf/h1_2_with_RH56DFTP_hands.urdf (robot description, URDF)
Before this commit: robot h1_2_with_RH56DFTP_hands, 58 links, 57 joints
Joints:
- joint left_index_1_joint: limit lower=0 upper=1.60795403606 effort=1 velocity=100 -> lower=0 upper=1.62 effort=1 velocity=100
- joint left_index_2_joint: limit lower=0 upper=1.68835173786 effort=1 velocity=100 -> lower=0 upper=1.377 effort=1 velocity=100; mimic joint=left_index_1_joint multiplier=1.05 offset=0 -> joint=left_index_1_joint multiplier=0.85 offset=0
- joint left_little_1_joint: limit lower=0 upper=1.67172785459 effort=1 velocity=100 -> lower=0 upper=1.62 effort=1 velocity=100
- joint left_little_2_joint: limit lower=0 upper=1.75531424732 effort=1 velocity=100 -> lower=0 upper=1.377 effort=1 velocity=100; mimic joint=left_little_1_joint multiplier=1.05 offset=0 -> joint=left_little_1_joint multiplier=0.85 offset=0
- joint left_middle_1_joint: limit lower=0 upper=1.590368352 effort=1 velocity=100 -> lower=0 upper=1.62 effort=1 velocity=100
- joint left_middle_2_joint: limit lower=0 upper=1.6698867696 effort=1 velocity=100 -> lower=0 upper=1.377 effort=1 velocity=100; mimic joint=left_middle_1_joint multiplier=1.05 offset=0 -> joint=left_middle_1_joint multiplier=0.85 offset=0
- joint left_ring_1_joint: limit lower=0 upper=1.60951229147 effort=1 velocity=100 -> lower=0 upper=1.62 effort=1 velocity=100
- joint left_ring_2_joint: limit lower=0 upper=1.68998790605 effort=1 velocity=100 -> lower=0 upper=1.377 effort=1 velocity=100; mimic joint=left_ring_1_joint multiplier=1.05 offset=0 -> joint=left_ring_1_joint multiplier=0.85 offset=0
- joint left_thumb_1_joint: limit lower=0 upper=1.06242095936 effort=1 velocity=100 -> lower=0 upper=0.66 effort=1 velocity=100
- joint left_thumb_2_joint: limit lower=0 upper=0.424968383745 effort=1 velocity=100 -> lower=0 upper=0.264 effort=1 velocity=100
- joint left_thumb_3_joint: limit lower=0 upper=0.637452575618 effort=1 velocity=100 -> lower=0 upper=0.396 effort=1 velocity=100
- joint left_thumb_swing_joint: limit lower=0 upper=1.30899614247 effort=1 velocity=100 -> lower=0 upper=1.19 effort=1 velocity=100
- joint right_index_1_joint: limit lower=0 upper=1.60795403606 effort=1 velocity=100 -> lower=0 upper=1.62 effort=1 velocity=100
- joint right_index_2_joint: limit lower=0 upper=1.68835173786 effort=1 velocity=100 -> lower=0 upper=1.377 effort=1 velocity=100; mimic joint=right_index_1_joint multiplier=1.05 offset=0 -> joint=right_index_1_joint multiplier=0.85 offset=0
- joint right_little_1_joint: limit lower=0 upper=1.67172785459 effort=1 velocity=100 -> lower=0 upper=1.62 effort=1 velocity=100
- joint right_little_2_joint: limit lower=0 upper=1.75531424732 effort=1 velocity=100 -> lower=0 upper=1.377 effort=1 velocity=100; mimic joint=right_little_1_joint multiplier=1.05 offset=0 -> joint=right_little_1_joint multiplier=0.85 offset=0
- joint right_middle_1_joint: limit lower=0 upper=1.590368352 effort=1 velocity=100 -> lower=0 upper=1.62 effort=1 velocity=100
- joint right_middle_2_joint: limit lower=0 upper=1.6698867696 effort=1 velocity=100 -> lower=0 upper=1.377 effort=1 velocity=100; mimic joint=right_middle_1_joint multiplier=1.05 offset=0 -> joint=right_middle_1_joint multiplier=0.85 offset=0
- joint right_ring_1_joint: limit lower=0 upper=1.60951229147 effort=1 velocity=100 -> lower=0 upper=1.62 effort=1 velocity=100
- joint right_ring_2_joint: limit lower=0 upper=1.68998790605 effort=1 velocity=100 -> lower=0 upper=1.377 effort=1 velocity=100; mimic joint=right_ring_1_joint multiplier=1.05 offset=0 -> joint=right_ring_1_joint multiplier=0.85 offset=0
- joint right_thumb_1_joint: limit lower=0 upper=1.06242095936 effort=1 velocity=100 -> lower=0 upper=0.66 effort=1 velocity=100
- joint right_thumb_2_joint: limit lower=0 upper=0.424968383745 effort=1 velocity=100 -> lower=0 upper=0.264 effort=1 velocity=100
- joint right_thumb_3_joint: limit lower=0 upper=0.637452575618 effort=1 velocity=100 -> lower=0 upper=0.396 effort=1 velocity=100
- joint right_thumb_swing_joint: limit lower=0 upper=1.30899614247 effort=1 velocity=100 -> lower=0 upper=1.19 effort=1 velocity=100

File: ros_h1_2_ws/src/h1_2_inspire_description/urdf/inspire_hand_left.urdf.xacro (robot description, xacro)
@@ -5,6 +5,6 @@
        left_index_1_joint, left_middle_1_joint, left_ring_1_joint, left_little_1_joint
      Mimic joints: left_thumb_2_joint (0.40×), left_thumb_3_joint (0.60×),
-       left_index_2_joint (1.05×), left_middle_2_joint (1.05×),
-       left_ring_2_joint (1.05×), left_little_2_joint (1.05×)
+       left_index_2_joint (0.85×), left_middle_2_joint (0.85×),
+       left_ring_2_joint (0.85×), left_little_2_joint (0.85×)
      Palm mass is set from a scale reading of the real hand: 0.840 kg for the
      whole hand, wrist flange included. The 12 digits keep their exported
@@ -16,22 +16,37 @@
      the tensor is scaled by 0.696619/0.314091 = 2.217891, which keeps the
      vendor's mass distribution. Both palms carry the same values, mirrored.
-     Joint zeros and limits follow the RH56DFTP user manual, section 2.6.11
-     (printed pages 21 and 22), which defines one chord angle per DOF against
-     the metacarpal plane. For every actuated joint q=0 is the hand FULLY OPEN
-     and the upper limit is FULLY CLOSED, so the SDK scale maps uniformly:
-       ANGLE_SET = 1000 * (1 - q / q_max)        q = q_max * (1 - ANGLE_SET/1000)
-     | DOF            | manual angle    | open  | closed | q_max (rad) |
-     | fingers        | alpha           | 176   | 20     | see below   |
-     | thumb bending  | theta           | 70    | -13    | 1.06242     |
-     | thumb rotation | beta            | 165   | 90     | 1.30900     |
-     q_max per finger: index 1.60795, middle 1.59037, ring 1.60951,
-     little 1.67173. They differ because each finger seats at its own angle on
-     the palm, so the same 176..20 sweep needs a slightly different joint
-     travel. The mimic joints carry multiplier * q_max.
-     Every joint origin was rotated so that q=0 lands exactly on the open
-     angle; the shifts were 0.4 to 1.9 degrees except thumb_swing, which moved
-     12.85 degrees. No joint axis was changed: all six close as q grows.
-     Verified by computing the manual's angles on this model: all twelve
-     endpoints land on target to better than 0.001 degrees. -->
+     q=0 is the hand FULLY OPEN and the upper limit is FULLY CLOSED on every
+     actuated joint, so all six close as q grows.
+     The ZEROS follow the RH56DFTP user manual, section 2.6.11 (printed pages
+     21 and 22), which defines one chord angle per DOF against the metacarpal
+     plane: alpha = 176 deg (fingers), theta = 70 deg (thumb bending) and
+     beta = 165 deg (thumb rotation) at ANGLE_SET = 1000. Every joint origin was
+     rotated so that q=0 lands on those angles. Photos of the real hand agree
+     to within about 3 deg (thumb rotation: 3 to 6 deg).
+     The UPPER LIMITS do not follow the manual: the real hand stops short of
+     the manual's closed angles. They were measured on photos of the real hand
+     at ANGLE_SET = 0, 500 and 1000 (inspire_hand_interface/Caracterizacion/
+     imagenes/angulos limite). This model was rendered in MuJoCo through a
+     virtual camera fitted to each photo, and the joint values were swept
+     until the rendered silhouette matched the photographed one.
+     | DOF            | q_max (rad) | real closed angle | manual closed |
+     | fingers        | 1.620       | alpha 31 to 37    | alpha 20      |
+     | thumb bending  | 0.660       | theta about 19    | theta -13     |
+     | thumb rotation | 1.190       | beta 96 to 97     | beta 90       |
+     The four fingers share one q_max that minimises the error over the four
+     photos (per finger 1.58 to 1.74). The finger mimic multiplier is 0.85,
+     not the vendor's 1.05, which folded the distal phalanx into the palm.
+     0.85 reproduces the closed pose to 0.5 deg of fingertip orientation. The
+     real coupling is not linear (about 0.65 at mid travel, 0.82 closed), so
+     at ANGLE_SET = 500 the modelled fingertip is about 13 deg too bent. The
+     thumb multipliers 0.40 and 0.60 cannot be resolved from the photos and
+     stay as exported.
+     The SDK scale is NOT linear in the finger proximal joints: at
+     ANGLE_SET = 500 they have already covered 64 percent of their travel.
+     Interpolate between the measured points, with s = 1 - ANGLE_SET/1000:
+     | s            | 0 | 0.5        | 1     |
+     | finger *_1   | 0 | 1.05       | 1.620 |
+     | thumb_1      | 0 | 0.38       | 0.660 |
+     | thumb_swing  | 0 | (no photo) | 1.190 |  -->
 <robot xmlns:xacro="http://www.ros.org/wiki/xacro">
   <link name="left_hand_base_link">
@@ -86,5 +101,5 @@
     <child link="left_thumb_swing"/>
     <axis xyz="0 0 1"/>
-    <limit lower="0" upper="1.30899614247" effort="1" velocity="100"/>
+    <limit lower="0" upper="1.19" effort="1" velocity="100"/>
   </joint>
   <link name="left_thumb_1">
@@ -116,5 +131,5 @@
     <child link="left_thumb_1"/>
     <axis xyz="0 0 -1"/>
-    <limit lower="0" upper="1.06242095936" effort="1" velocity="100"/>
+    <limit lower="0" upper="0.66" effort="1" velocity="100"/>
   </joint>
   <link name="left_thumb_2">
@@ -146,5 +161,5 @@
     <child link="left_thumb_2"/>
     <axis xyz="0 0 -1"/>
-    <limit lower="0" upper="0.424968383745" effort="1" velocity="100"/>
+    <limit lower="0" upper="0.264" effort="1" velocity="100"/>
     <mimic joint="left_thumb_1_joint" multiplier="0.40" offset="0"/>
   </joint>
@@ -177,5 +192,5 @@
     <child link="left_thumb_3"/>
     <axis xyz="0 0 -1"/>
-    <limit lower="0" upper="0.637452575618" effort="1" velocity="100"/>
+    <limit lower="0" upper="0.396" effort="1" velocity="100"/>
     <mimic joint="left_thumb_1_joint" multiplier="0.60" offset="0"/>
   </joint>
@@ -208,5 +223,5 @@
     <child link="left_index_1"/>
     <axis xyz="0 0 -1"/>
-    <limit lower="0" upper="1.60795403606" effort="1" velocity="100"/>
+    <limit lower="0" upper="1.62" effort="1" velocity="100"/>
   </joint>
   <link name="left_index_2">
@@ -238,6 +253,6 @@
     <child link="left_index_2"/>
     <axis xyz="0 0 -1"/>
-    <limit lower="0" upper="1.68835173786" effort="1" velocity="100"/>
-    <mimic joint="left_index_1_joint" multiplier="1.05" offset="0"/>
+    <limit lower="0" upper="1.377" effort="1" velocity="100"/>
+    <mimic joint="left_index_1_joint" multiplier="0.85" offset="0"/>
   </joint>
   <link name="left_middle_1">
@@ -269,5 +284,5 @@
     <child link="left_middle_1"/>
     <axis xyz="0 0 -1"/>
-    <limit lower="0" upper="1.590368352" effort="1" velocity="100"/>
+    <limit lower="0" upper="1.62" effort="1" velocity="100"/>
   </joint>
   <link name="left_middle_2">
@@ -299,6 +314,6 @@
     <child link="left_middle_2"/>
     <axis xyz="0 0 -1"/>
-    <limit lower="0" upper="1.6698867696" effort="1" velocity="100"/>
-    <mimic joint="left_middle_1_joint" multiplier="1.05" offset="0"/>
+    <limit lower="0" upper="1.377" effort="1" velocity="100"/>
+    <mimic joint="left_middle_1_joint" multiplier="0.85" offset="0"/>
   </joint>
   <link name="left_ring_1">
@@ -330,5 +345,5 @@
     <child link="left_ring_1"/>
     <axis xyz="0 0 -1"/>
-    <limit lower="0" upper="1.60951229147" effort="1" velocity="100"/>
+    <limit lower="0" upper="1.62" effort="1" velocity="100"/>
   </joint>
   <link name="left_ring_2">
@@ -360,6 +375,6 @@
     <child link="left_ring_2"/>
     <axis xyz="0 0 -1"/>
-    <limit lower="0" upper="1.68998790605" effort="1" velocity="100"/>
-    <mimic joint="left_ring_1_joint" multiplier="1.05" offset="0"/>
+    <limit lower="0" upper="1.377" effort="1" velocity="100"/>
+    <mimic joint="left_ring_1_joint" multiplier="0.85" offset="0"/>
   </joint>
   <link name="left_little_1">
@@ -391,5 +406,5 @@
     <child link="left_little_1"/>
     <axis xyz="0 0 -1"/>
-    <limit lower="0" upper="1.67172785459" effort="1" velocity="100"/>
+    <limit lower="0" upper="1.62" effort="1" velocity="100"/>
   </joint>
   <link name="left_little_2">
@@ -421,6 +436,6 @@
     <child link="left_little_2"/>
     <axis xyz="0 0 -1"/>
-    <limit lower="0" upper="1.75531424732" effort="1" velocity="100"/>
-    <mimic joint="left_little_1_joint" multiplier="1.05" offset="0"/>
+    <limit lower="0" upper="1.377" effort="1" velocity="100"/>
+    <mimic joint="left_little_1_joint" multiplier="0.85" offset="0"/>
   </joint>
 </robot>
